File: Test_board_BAKALARKA/test_board.kicad_pcb (KiCad board)
At the start: 2 copper layers, 30 parts, among them J1 USB_C_Receptacle_USB2.0_16P, SW1 SW_SPST, SW2 SW_SPST, U1 LM27762, U2 ESP32-S3-WROOM-2, U3 HT75xx-1-SOT89

Commit message: pridani textu peak detect, xor phase, signal source
Parts:
- added ADC1: NCD98011, Package_DFN_QFN:Texas_UQFN-8_1.5x1.5mm_P0.5mm, F.Cu at (243.8, 274.6)
- added ADC2: NCD98011, Package_DFN_QFN:Texas_UQFN-8_1.5x1.5mm_P0.5mm, F.Cu at (245.1, 317.8)
- added C13: 100n, Capacitor_SMD:C_0603_1608Metric_Pad1.08x0.95mm_HandSolder, F.Cu at (373.4, 377.5)
- added C14: 100n, Capacitor_SMD:C_0603_1608Metric_Pad1.08x0.95mm_HandSolder, F.Cu at (15.2, 391.4)
- added C15: 100n, Capacitor_SMD:C_0603_1608Metric_Pad1.08x0.95mm_HandSolder, F.Cu at (395.0, 377.5)
- added C16: 100n, Capacitor_SMD:C_0603_1608Metric_Pad1.08x0.95mm_HandSolder, F.Cu at (50.8, 399.1)
- added C17: 100n, Capacitor_SMD:C_0603_1608Metric_Pad1.08x0.95mm_HandSolder, F.Cu at (73.7, 402.9)
- added C18: 330n, Capacitor_SMD:C_0603_1608Metric_Pad1.08x0.95mm_HandSolder, F.Cu at (68.6, 282.2)
- added C19: 330n, Capacitor_SMD:C_0603_1608Metric_Pad1.08x0.95mm_HandSolder, F.Cu at (80.0, 282.2)
- added C20: 330n, Capacitor_SMD:C_0603_1608Metric_Pad1.08x0.95mm_HandSolder, F.Cu at (69.8, 347.0)
- added C21: 330n, Capacitor_SMD:C_0603_1608Metric_Pad1.08x0.95mm_HandSolder, F.Cu at (81.3, 347.0)
- added C22: 330n, Capacitor_SMD:C_0603_1608Metric_Pad1.08x0.95mm_HandSolder, F.Cu at (86.4, 319.1)
- added C23: 330n, Capacitor_SMD:C_0603_1608Metric_Pad1.08x0.95mm_HandSolder, F.Cu at (91.4, 303.8)
- added C24: 100n, Capacitor_SMD:C_0603_1608Metric_Pad1.08x0.95mm_HandSolder, F.Cu at (395.0, 402.9)
- added C25: 100n, Capacitor_SMD:C_0603_1608Metric_Pad1.08x0.95mm_HandSolder, F.Cu at (221.0, 352.1)
- added C26: 100n, Capacitor_SMD:C_0603_1608Metric_Pad1.08x0.95mm_HandSolder, F.Cu at (373.4, 402.9)
- added C27: 100n, Capacitor_SMD:C_0603_1608Metric_Pad1.08x0.95mm_HandSolder, F.Cu at (221.0, 377.5)
- added C28: 100n, Capacitor_SMD:C_0603_1608Metric_Pad1.08x0.95mm_HandSolder, F.Cu at (105.4, 405.4)
- added C29: 100n, Capacitor_SMD:C_0603_1608Metric_Pad1.08x0.95mm_HandSolder, F.Cu at (199.4, 352.1)
- added C30: 100n, Capacitor_SMD:C_0603_1608Metric_Pad1.08x0.95mm_HandSolder, F.Cu at (199.4, 377.5)
- added C31: 100n, Capacitor_SMD:C_0603_1608Metric_Pad1.08x0.95mm_HandSolder, F.Cu at (254.0, 297.5)
- added C32: 100n, Capacitor_SMD:C_0603_1608Metric_Pad1.08x0.95mm_HandSolder, F.Cu at (254.0, 306.4)
- added C33: 100n, Capacitor_SMD:C_0603_1608Metric_Pad1.08x0.95mm_HandSolder, F.Cu at (252.7, 253.0)
- added C34: 100n, Capacitor_SMD:C_0603_1608Metric_Pad1.08x0.95mm_HandSolder, F.Cu at (252.7, 261.9)
- added C35: 1u, Capacitor_SMD:C_0603_1608Metric_Pad1.08x0.95mm_HandSolder, F.Cu at (160.0, 325.4)
- added C36: 1u, Capacitor_SMD:C_0603_1608Metric_Pad1.08x0.95mm_HandSolder, F.Cu at (143.5, 279.7)
- added C37: 100n, Capacitor_SMD:C_0603_1608Metric_Pad1.08x0.95mm_HandSolder, F.Cu at (83.2, 37.7)
- added C38: 100n, Capacitor_SMD:C_0603_1608Metric_Pad1.08x0.95mm_HandSolder, F.Cu at (79.7, 37.7)
- added C39: 330n, Capacitor_SMD:C_0603_1608Metric_Pad1.08x0.95mm_HandSolder, F.Cu at (90.2, 239.1)
- added C40: 330n, Capacitor_SMD:C_0603_1608Metric_Pad1.08x0.95mm_HandSolder, F.Cu at (85.1, 254.3)
- added J2: Conn_Coaxial, Connector_Coaxial:BNC_Amphenol_B6252HB-NPP3G-50_Horizontal, F.Cu at (125.7, 121.9)
- added J3: Conn_Coaxial, Connector_Coaxial:BNC_Amphenol_B6252HB-NPP3G-50_Horizontal, F.Cu at (109.4, 121.9)
- added JP1: Jumper_3_Open, Connector_PinHeader_2.54mm:PinHeader_1x03_P2.54mm_Vertical, F.Cu at (36.8, 265.7)
- added JP10: SolderJumper_3_Open, Jumper:SolderJumper-3_P1.3mm_Open_RoundedPad1.0x1.5mm, F.Cu at (73.5, 47.0)
- added JP11: SolderJumper_3_Open, Jumper:SolderJumper-3_P1.3mm_Open_RoundedPad1.0x1.5mm, F.Cu at (73.5, 52.0)
- added JP2: Jumper_3_Open, Connector_PinHeader_2.54mm:PinHeader_1x03_P2.54mm_Vertical, F.Cu at (45.7, 278.4)
- added JP3: Jumper_3_Open, Connector_PinHeader_2.54mm:PinHeader_1x03_P2.54mm_Vertical, F.Cu at (129.5, 334.3)
- added JP4: Jumper_2_Open, Connector_PinHeader_1.00mm:PinHeader_1x02_P1.00mm_Vertical, F.Cu at (184.2, 312.7)
- added JP5: Jumper_3_Open, Connector_PinHeader_2.54mm:PinHeader_1x03_P2.54mm_Vertical, F.Cu at (128.3, 265.7)
- added JP6: Jumper_2_Open, Connector_PinHeader_1.00mm:PinHeader_1x02_P1.00mm_Vertical, F.Cu at (180.3, 274.6)
- added JP7: SolderJumper_3_Open, Jumper:SolderJumper-3_P1.3mm_Open_RoundedPad1.0x1.5mm, F.Cu at (269.2, 305.1)
- added JP8: SolderJumper_3_Open, Jumper:SolderJumper-3_P1.3mm_Open_RoundedPad1.0x1.5mm, F.Cu at (269.2, 317.8)
- added JP9: SolderJumper_3_Open, Jumper:SolderJumper-3_P1.3mm_Open_RoundedPad1.0x1.5mm, F.Cu at (269.2, 330.5)
- added Q1: NX3008NBK, Package_TO_SOT_SMD:SOT-323_SC-70_Handsoldering, F.Cu at (256.5, 353.4)
- added R12: 10k, Resistor_SMD:R_0603_1608Metric_Pad0.98x0.95mm_HandSolder, F.Cu at (200.7, 284.8)
- added R13: 10k, Resistor_SMD:R_0603_1608Metric_Pad0.98x0.95mm_HandSolder, F.Cu at (66.0, 402.9)
- added R14: 10k, Resistor_SMD:R_0603_1608Metric_Pad0.98x0.95mm_HandSolder, F.Cu at (83.8, 286.0)
- added R15: 10k, Resistor_SMD:R_0603_1608Metric_Pad0.98x0.95mm_HandSolder, F.Cu at (88.9, 270.8)
- added R16: 10k, Resistor_SMD:R_0603_1608Metric_Pad0.98x0.95mm_HandSolder, F.Cu at (71.1, 315.2)
- added R17: 10k, Resistor_SMD:R_0603_1608Metric_Pad0.98x0.95mm_HandSolder, F.Cu at (82.5, 315.2)
- added R18: 10k, Resistor_SMD:R_0603_1608Metric_Pad0.98x0.95mm_HandSolder, F.Cu at (85.1, 350.8)
- added R19: 10k, Resistor_SMD:R_0603_1608Metric_Pad0.98x0.95mm_HandSolder, F.Cu at (90.2, 335.6)
- added R20: 10k, Resistor_SMD:R_0603_1608Metric_Pad0.98x0.95mm_HandSolder, F.Cu at (212.1, 279.7)
- added R21: 10k, Resistor_SMD:R_0603_1608Metric_Pad0.98x0.95mm_HandSolder, F.Cu at (191.8, 261.9)
- added R22: 10k, Resistor_SMD:R_0603_1608Metric_Pad0.98x0.95mm_HandSolder, F.Cu at (191.8, 269.5)
- added R23: 10k, Resistor_SMD:R_0603_1608Metric_Pad0.98x0.95mm_HandSolder, F.Cu at (193.0, 305.1)
- added R24: 10k, Resistor_SMD:R_0603_1608Metric_Pad0.98x0.95mm_HandSolder, F.Cu at (193.0, 312.7)
- added R25: 10k, Resistor_SMD:R_0603_1608Metric_Pad0.98x0.95mm_HandSolder, F.Cu at (201.9, 327.9)
- added R26: 10k, Resistor_SMD:R_0603_1608Metric_Pad0.98x0.95mm_HandSolder, F.Cu at (213.4, 322.9)
- added R27: 4k7, Resistor_SMD:R_0603_1608Metric_Pad0.98x0.95mm_HandSolder, F.Cu at (259.1, 344.5)
- added R35: 10k, Resistor_SMD:R_0603_1608Metric_Pad0.98x0.95mm_HandSolder, F.Cu at (81.3, 250.5)
- added R36: 10k, Resistor_SMD:R_0603_1608Metric_Pad0.98x0.95mm_HandSolder, F.Cu at (69.8, 250.5)
- added R7: 10k, Resistor_SMD:R_0603_1608Metric_Pad0.98x0.95mm_HandSolder, F.Cu at (66.0, 395.3)
- added TP1: TestPoint, Connector_Pin:Pin_D1.3mm_L11.0mm_LooseFit, F.Cu at (130.2, 45.2)
- added TP2: TestPoint, Connector_Pin:Pin_D1.3mm_L11.0mm_LooseFit, F.Cu at (130.2, 49.8)
- added TP3: TestPoint, Connector_Pin:Pin_D1.3mm_L11.0mm_LooseFit, F.Cu at (47.8, 47.2)
- added TP4: TestPoint, Connector_Pin:Pin_D1.3mm_L11.0mm_LooseFit, F.Cu at (130.2, 40.8)
- added TP4: TestPoint, Connector_Pin:Pin_D1.3mm_L11.0mm_LooseFit, F.Cu at (52.8, 47.2)
- added U11: REF3033, Package_TO_SOT_SMD:SOT-23, F.Cu at (38.1, 391.4)
- added U20: CD74HC4052, Package_SO:TSSOP-16_4.4x5mm_P0.65mm, F.Cu at (161.3, 298.7)
- added U4: TL074, Package_SO:TSSOP-14_4.4x5mm_P0.65mm, F.Cu at (219.7, 364.8)
- added U5: TL074, Package_SO:TSSOP-14_4.4x5mm_P0.65mm, F.Cu at (101.6, 253.0)
- added U6: CH340G, Package_SO:SOIC-16_3.9x9.9mm_P1.27mm, F.Cu at (81.6, 49.5)
- added Y1: 12MHz, Crystal:Crystal_SMD_HC49-SD_HandSoldering, F.Cu at (81.2, 41.7)
- moved R7 325.0 mm to (66.0, 395.3), turned to 180 degrees
- moved R4 157.9 mm to (41.8, 52.5), turned to -90 degrees
- moved U3 151.9 mm to (43.0, 42.5), turned to 90 degrees
- moved D1 147.9 mm to (47.0, 39.5), turned to -90 degrees
- moved SW1 147.1 mm to (38.8, 55.8), turned to -90 degrees
- moved R6 140.9 mm to (59.2, 48.5)
- moved C3 139.0 mm to (39.5, 44.0), turned to -90 degrees
- moved R11 135.9 mm to (49.0, 39.5), turned to 90 degrees
- moved C8 135.1 mm to (43.5, 49.0), turned to 180 degrees
- moved C2 135.0 mm to (43.5, 47.5), turned to 180 degrees
- moved R5 130.9 mm to (69.0, 68.5), turned to 90 degrees
- moved J1 128.7 mm to (58.0, 39.8), turned to 180 degrees
- moved R9 116.6 mm to (65.5, 38.0), turned to 90 degrees
- moved R8 114.5 mm to (67.0, 38.0), turned to 90 degrees
- moved SW2 109.6 mm to (72.2, 70.8), turned to 90 degrees
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Connections:
- U2 pad 13: /USB+Power/USB- -> Net-(JP11-C)
- U2 pad 14: /USB+Power/USB+ -> Net-(JP10-C)
- U2 pad 15: unconnected-(U1-GPIO3/TOUCH3/ADC1_CH2-Pad15) -> /Analog/~{CS_{1}}
- U2 pad 36: unconnected-(U1-U0RXD/GPIO44/CLK_OUT2-Pad36) -> Net-(U2-U0RXD/GPIO44/CLK_OUT2)
- U2 pad 37: unconnected-(U1-U0TXD/GPIO43/CLK_OUT1-Pad37) -> Net-(U2-U0TXD/GPIO43/CLK_OUT1)
- U2 pad 38: unconnected-(U1-GPIO2/TOUCH2/ADC1_CH1-Pad38) -> /Analog/ADC_DATA_{1}
- U2 pad 39: unconnected-(U1-GPIO1/TOUCH1/ADC1_CH0-Pad39) -> /Analog/ADC_CLK_{1}
- U2 pad 4: unconnected-(U1-GPIO4/TOUCH4/ADC1_CH3-Pad4) -> /Analog/ADC_CLK_{2}
- U2 pad 5: unconnected-(U1-GPIO5/TOUCH5/ADC1_CH4-Pad5) -> /Analog/ADC_DATA_{2}
- U2 pad 6: unconnected-(U1-GPIO6/TOUCH6/ADC1_CH5-Pad6) -> /Analog/~{CS_{2}}
Routing:
- net +5V_USB: track 0.00 -> 120.1 mm, vias 0 -> 10
- net GND: track 0.00 -> 117.7 mm, vias 0 -> 15
- net Net-(U2-U0TXD/GPIO43/CLK_OUT1): track 0.00 -> 98.9 mm, vias 0 -> 2
- net Net-(U2-U0RXD/GPIO44/CLK_OUT2): track 0.00 -> 94.1 mm, vias 0 -> 2
- net +3V3: track 0.00 -> 50.7 mm, vias 0 -> 2
- net +5V: track 0.00 -> 34.0 mm, vias 0 -> 2
- net -5V: track 0.00 -> 29.0 mm, vias 0 -> 1
- net /USB+Power/USB-: track 0.00 -> 22.9 mm
- net /USB+Power/USB+: track 0.00 -> 21.9 mm
- net Net-(U6-XI): track 0.00 -> 13.9 mm
- net Net-(JP10-C): track 0.00 -> 13.3 mm, vias 0 -> 2
- net Net-(SW1-B): track 0.00 -> 12.3 mm
- net Net-(JP11-C): track 0.00 -> 12.1 mm
- net Net-(J1-CC2): track 0.00 -> 12.1 mm
- net Net-(JP10-A): track 0.00 -> 11.0 mm
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- added copper zone on B.Cu, net GND
Other:
- board outline added: 99.9 x 99.9 mm
- board text added: "Analog"

Commit message: fix citace a uvod
Parts:
- removed C26: 100n, Capacitor_SMD:C_0603_1608Metric_Pad1.08x0.95mm_HandSolder
- removed the R7 at (66.0, 395.3)
- removed the TP4 at (52.8, 47.2)
- added D2: XINGLIGHT XL-1615RGBC-2812B-S, Snapeda:XINGLIGHT XL-1615RGBC-2812B-S, F.Cu at (41.4, 63.5)
- added D3: XINGLIGHT XL-1615RGBC-2812B-S, Snapeda:XINGLIGHT XL-1615RGBC-2812B-S, F.Cu at (38.8, 63.5)
- added J4: Conn_Coaxial, Snapeda:BNC_Gold, F.Cu at (129.2, 106.7)
- added R28: 10k, Resistor_SMD:R_0603_1608Metric_Pad0.98x0.95mm_HandSolder, F.Cu at (115.9, 69.2)
- added R29: 10k, Resistor_SMD:R_0603_1608Metric_Pad0.98x0.95mm_HandSolder, F.Cu at (115.9, 65.8)
- added TP10: TestPoint, Connector_Pin:Pin_D1.0mm_L10.0mm, F.Cu at (94.9, 103.2)
- added TP11: TestPoint, Connector_Pin:Pin_D1.0mm_L10.0mm, F.Cu at (100.7, 71.6)
- added TP12: TestPoint, Connector_Pin:Pin_D1.0mm_L10.0mm, F.Cu at (100.7, 82.0)
- added TP13: TestPoint, Connector_Pin:Pin_D1.0mm_L10.0mm, F.Cu at (74.5, 88.6)
- added TP14: TestPoint, Connector_Pin:Pin_D1.0mm_L10.0mm, F.Cu at (74.5, 94.6)
- added TP15: TestPoint, Connector_Pin:Pin_D1.3mm_L11.0mm_LooseFit, F.Cu at (100.7, 76.8)
- added TP16: TestPoint, Connector_Pin:Pin_D1.3mm_L11.0mm_LooseFit, F.Cu at (57.1, 88.8)
- added TP17: TestPoint, Connector_Pin:Pin_D1.3mm_L11.0mm_LooseFit, F.Cu at (71.1, 98.0)
- added TP18: TestPoint, Connector_Pin:Pin_D1.3mm_L11.0mm_LooseFit, F.Cu at (83.1, 128.2)
- added TP19: TestPoint, Connector_Pin:Pin_D1.3mm_L11.0mm_LooseFit, F.Cu at (52.1, 47.9)
- added TP20: TestPoint, Connector_Pin:Pin_D1.0mm_L10.0mm, F.Cu at (112.7, 69.2)
- added TP21: TestPoint, Connector_Pin:Pin_D1.0mm_L10.0mm, F.Cu at (127.7, 69.0)
- added TP22: TestPoint, Connector_Pin:Pin_D1.0mm_L10.0mm, F.Cu at (112.7, 65.0)
- added TP23: TestPoint, Connector_Pin:Pin_D1.0mm_L10.0mm, F.Cu at (127.8, 65.2)
- added TP5: TestPoint, Connector_Pin:Pin_D1.0mm_L10.0mm, F.Cu at (60.3, 123.2)
- added TP6: TestPoint, Connector_Pin:Pin_D1.0mm_L10.0mm, F.Cu at (77.7, 123.2)
- added TP7: TestPoint, Connector_Pin:Pin_D1.0mm_L10.0mm, F.Cu at (88.7, 123.2)
- added TP8: TestPoint, Connector_Pin:Pin_D1.0mm_L10.0mm, F.Cu at (107.3, 123.2)
- added TP9: TestPoint, Connector_Pin:Pin_D1.0mm_L10.0mm, F.Cu at (73.1, 103.5)
- added U7: OPA2810, Package_SO:SOIC-8_3.9x4.9mm_P1.27mm, F.Cu at (121.6, 67.1)
- added kibuzzard-69579972: G***, kibuzzard-69579972, F.Cu at (106.3, 115.0)
- added kibuzzard-69579972: G***, kibuzzard-69579972, F.Cu at (70.9, 115.0)
- added kibuzzard-695799A4: G***, kibuzzard-695799A4, F.Cu at (96.9, 115.0)
- added kibuzzard-695799A4: G***, kibuzzard-695799A4, F.Cu at (61.5, 115.0)
- added kibuzzard-6957FD09: G***, kibuzzard-6957FD09, F.Cu at (107.1, 71.4)
- added kibuzzard-6957FD1B: G***, kibuzzard-6957FD1B, F.Cu at (107.1, 82.0)
- added kibuzzard-6958001D: G***, kibuzzard-6958001D, F.Cu at (105.9, 76.8)
- added kibuzzard-6958001D: G***, kibuzzard-6958001D, F.Cu at (83.1, 131.2)
- added kibuzzard-6958001D: G***, kibuzzard-6958001D, F.Cu at (55.9, 92.0)
- added kibuzzard-6958001D: G***, kibuzzard-6958001D, F.Cu at (67.1, 100.2)
- added kibuzzard-69592FE8: G***, kibuzzard-69592FE8, F.Cu at (126.1, 71.6)
- added kibuzzard-69592FF5: G***, kibuzzard-69592FF5, F.Cu at (126.3, 61.8)
- C13: value 100n -> 4.7u; footprint Capacitor_SMD:C_0603_1608Metric_Pad1.08x0.95mm_HandSolder -> Capacitor_SMD:C_0805_2012Metric_Pad1.18x1.45mm_HandSolder
- C37, C38: value 100n -> 22p
- JP4, JP6: footprint Connector_PinHeader_1.00mm:PinHeader_1x02_P1.00mm_Vertical -> Connector_PinHeader_2.54mm:PinHeader_1x02_P2.54mm_Vertical
- R7: value R_Small -> 10k
- moved C13 434.0 mm to (66.7, 70.4), turned to 0 degrees
- moved C24 431.3 mm to (120.0, 70.6), turned to 180 degrees
- moved C15 415.2 mm to (123.3, 63.5), turned to 0 degrees
- moved Q1 338.9 mm to (54.9, 81.0), turned to 180 degrees
- moved R27 331.7 mm to (54.7, 83.2), turned to 180 degrees
- moved C16 330.8 mm to (93.5, 71.0), turned to -90 degrees
- moved C14 328.6 mm to (88.3, 71.1), turned to -90 degrees
- moved JP9 327.3 mm to (52.3, 85.4), turned to 0 degrees
- moved R13 326.5 mm to (89.2, 77.2), turned to 0 degrees
- moved U11 324.9 mm to (90.8, 70.9), turned to 90 degrees
- moved C17 324.5 mm to (89.2, 78.8), turned to 0 degrees
- moved C28 324.4 mm to (95.1, 81.2), turned to -90 degrees
- moved JP8 322.9 mm to (42.6, 87.8), turned to 0 degrees
- moved C27 320.1 mm to (87.2, 86.7), turned to 90 degrees
- moved R7 319.2 mm to (92.6, 77.2), turned to 0 degrees
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Connections:
- C13 pad 1: GND -> +3V3
- C13 pad 2: +5V -> GND
- JP10 pad 2: Net-(JP10-C) -> /USB+Power/USB+
- JP10 pad 3: /USB+Power/USB+ -> Net-(JP10-B)
- JP11 pad 2: Net-(JP11-C) -> /USB+Power/USB-
- JP11 pad 3: /USB+Power/USB- -> Net-(JP11-B)
- R7 pad 1: unconnected-(R1-Pad1) -> Net-(U4A-+)
- R7 pad 2: unconnected-(R1-Pad2) -> +3.3 V_{ref}
- U2 pad 12: unconnected-(U2-GPIO8/TOUCH8/ADC1_CH7/SUBSPICS1-Pad12) -> /Analog/Sw_B
- U2 pad 13: Net-(JP11-C) -> Net-(JP11-A)
- U2 pad 14: Net-(JP10-C) -> Net-(JP10-A)
- U2 pad 22: unconnected-(U2-GPIO14/TOUCH14/ADC2_CH3/FSPIWP/FSPIDQS/SUBSPIWP-Pad22) -> /additions/DIN_LED
- U2 pad 7: unconnected-(U2-GPIO7/TOUCH7/ADC1_CH6-Pad7) -> /Analog/Sw_A
- U20 pad 10: unconnected-(U20-A-Pad10) -> /Analog/Sw_A
- U20 pad 9: unconnected-(U20-B-Pad9) -> /Analog/Sw_B
- U6 pad 5: Net-(JP10-A) -> Net-(JP11-B)
- U6 pad 6: Net-(JP11-A) -> Net-(JP10-B)
Routing:
- net GND: track 117.7 -> 308.1 mm, vias 15 -> 63
- net +5V: track 34.0 -> 173.1 mm, vias 2 -> 7
- net -5V: track 29.0 -> 156.5 mm, vias 1 -> 4
- net +3V3: track 50.7 -> 176.9 mm, vias 2 -> 8
- net +3.3 V_{ref}: track 0.00 -> 72.3 mm, vias 0 -> 3
- net Net-(J2-In): track 0.00 -> 66.3 mm
- net /Analog/Sw_B: track 0.00 -> 63.1 mm, vias 0 -> 2
- net Net-(J3-In): track 0.00 -> 61.2 mm
- net /Analog/V_HighPass: track 0.00 -> 59.5 mm
- net /Analog/Sw_A: track 0.00 -> 59.3 mm, vias 0 -> 2
- net /Analog/I_LowPass: track 0.00 -> 56.2 mm
- net /Analog/ADC_CLK_{2}: track 0.00 -> 52.6 mm, vias 0 -> 2
- net /Analog/~{CS_{1}}: track 0.00 -> 48.2 mm, vias 0 -> 2
- net Net-(JP5-C): track 0.00 -> 42.5 mm
- net /Analog/V_LowPass: track 0.00 -> 41.6 mm, vias 0 -> 2
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Other:
- outline, holes or cut-outs redrawn
- board text added: "<-- Print test lines even if resolution too small"
- board text added: "CH340G"
- board text added: "Native"
- board text added: "Separate"
- board text added: "Shared"
- board text removed: "Analog"

Commit message: testboard frontpanel
Parts:
- removed kibuzzard-69579972 (x2): G***, kibuzzard-69579972
- removed kibuzzard-695799A4 (x2): G***, kibuzzard-695799A4
- removed kibuzzard-6957FD09: G***, kibuzzard-6957FD09
- removed kibuzzard-6957FD1B: G***, kibuzzard-6957FD1B
- removed the kibuzzard-6958001D at (105.9, 76.8)
- removed the kibuzzard-6958001D at (67.1, 100.2)
- removed kibuzzard-69592FE8: G***, kibuzzard-69592FE8
- removed kibuzzard-69592FF5: G***, kibuzzard-69592FF5
- added G***: LOGO, LOGO, F.Cu at (44.5, 105.0)
- added kibuzzard-696656D5: G***, kibuzzard-696656D5, F.Cu at (61.3, 115.0)
- added kibuzzard-696656FC: G***, kibuzzard-696656FC, F.Cu at (70.9, 115.0)
- added kibuzzard-69665706: G***, kibuzzard-69665706, F.Cu at (67.1, 100.2)
- added kibuzzard-69665710: G***, kibuzzard-69665710, F.Cu at (107.1, 82.0)
- added kibuzzard-69665718: G***, kibuzzard-69665718, F.Cu at (107.1, 71.4)
- added kibuzzard-6966571E: G***, kibuzzard-6966571E, F.Cu at (105.9, 76.8)
- added kibuzzard-69665729: G***, kibuzzard-69665729, F.Cu at (96.8, 115.0)
- added kibuzzard-69665736: G***, kibuzzard-69665736, F.Cu at (106.4, 115.0)
- added kibuzzard-6966573E: G***, kibuzzard-6966573E, F.Cu at (126.3, 61.8)
- added kibuzzard-69665743: G***, kibuzzard-69665743, F.Cu at (126.1, 71.6)
- added kibuzzard-696658C9: G***, kibuzzard-696658C9, B.Cu at (116.0, 101.0)
- added kibuzzard-696658E8: G***, kibuzzard-696658E8, B.Cu at (116.0, 103.5)
- added kibuzzard-696658F1: G***, kibuzzard-696658F1, B.Cu at (116.0, 106.0)
- added kibuzzard-696658F7: G***, kibuzzard-696658F7, B.Cu at (116.0, 108.5)
- added kibuzzard-696658FF: G***, kibuzzard-696658FF, B.Cu at (116.0, 111.0)
- added kibuzzard-69665908: G***, kibuzzard-69665908, B.Cu at (116.0, 113.5)
- added kibuzzard-6966592B: G***, kibuzzard-6966592B, B.Cu at (116.0, 116.0)
- added kibuzzard-6966594C: G***, kibuzzard-6966594C, B.Cu at (116.0, 117.5)
- added kibuzzard-69665967: G***, kibuzzard-69665967, B.Cu at (116.0, 118.5)
- added kibuzzard-69665B05: G***, kibuzzard-69665B05, F.Cu at (126.8, 45.2)
- added kibuzzard-69665B09: G***, kibuzzard-69665B09, F.Cu at (126.8, 49.8)
- added kibuzzard-69665B11: G***, kibuzzard-69665B11, F.Cu at (126.8, 40.6)
- J4: moved to B.Cu
- moved J4 0.30 mm to (129.2, 107.0), turned to 90 degrees
Routing:
- net unconnected-(J4-In-Pad1): track 0.00 -> 32.5 mm
- net GND: track 308.1 -> 315.7 mm, vias 63 -> 65
- net (no net): track 4.44 -> 0.00 mm, vias 2 -> 0
- net /Analog/I_LowPass: track 56.2 -> 55.5 mm
Other:
- board text added: "Design: Vojtěch Glombíček"
