File: Test_board_BAKALARKA/analog.kicad_sch (KiCad schematic)
At the start: 54 parts, among them J2 Conn_Coaxial, J3 Conn_Coaxial, U10 TL072, U11 REF3033, U20 CD74HC4052, U4 TL072, U6 TL072, U7 TL072, U8 TL072, U9 TL072

Commit message: pridani textu peak detect, xor phase, signal source
Parts:
- removed U10, U4, U6, U7, U8, U9: TL072, Package_SO:SOIC-8_3.9x4.9mm_P1.27mm, symbol Amplifier_Operational:TL072
- added C31, C32, C33, C34: 100n, Capacitor_SMD:C_0603_1608Metric_Pad1.08x0.95mm_HandSolder, symbol Device:C_Small
- added JP3, JP5: Jumper_3_Open, Connector_PinHeader_2.54mm:PinHeader_1x03_P2.54mm_Vertical, symbol Jumper:Jumper_3_Open
- added JP4, JP6: Jumper_2_Open, Connector_PinHeader_1.00mm:PinHeader_1x02_P1.00mm_Vertical, symbol Jumper:Jumper_2_Open
- added JP7, JP8, JP9: SolderJumper_3_Open, Jumper:SolderJumper-3_P1.3mm_Open_RoundedPad1.0x1.5mm, symbol Jumper:SolderJumper_3_Open
- added Q1: NX3008NBK, Package_TO_SOT_SMD:SOT-323_SC-70_Handsoldering, symbol Device:Q_NMOS_GSD
- added R27: 4k7, Resistor_SMD:R_0603_1608Metric_Pad0.98x0.95mm_HandSolder, symbol Device:R
- added U4, U5: TL074, Package_SO:TSSOP-14_4.4x5mm_P0.65mm, symbol Amplifier_Operational:TL074
Connections:
- net +1.65 V_{ref}: now also U4.1, U4.2 (-)
- net +3.3 V_{ref}: now also ADC1.6 (V_{REF}), ADC2.6 (V_{REF}), C31.1, C33.1
- net +3V3: now also ADC2.4 (V_{DD}), C32.1, C34.1, R27.1
- net +5V: now also U4.4 (V+), U5.4 (V+)
- net -5V: now also U4.11 (V-), U5.11 (V-)
- net GND: now also ADC1.5 (GND), ADC1.8 (IN-), ADC2.5 (GND), ADC2.8 (IN-), C31.2, C32.2, C33.2, C34.2, Q1.2 (S)
- net I_HighPass: now also JP3.1 (A), U5.13 (-), U5.14
- net I_LowPass: now also JP3.3 (B), U5.8, U5.9 (-)
- net V_HighPass: now also JP5.1 (A), U5.6 (-), U5.7
- net V_LowPass: now also JP5.3 (B), U5.1, U5.2 (-)
- net at R23.1, R24.1: now also U4.12 (+)
- net at C17.2, R13.2, R7.1: now also U4.3 (+)
- net at C40.1, R35.2: now also U5.3 (+)
- net at R21.1, R22.1: now also U4.10 (+)
- net at C22.1, R17.2: now also U5.10 (+)
- net at R24.2: now also JP3.2 (C), JP4.2 (B); no longer U20.3 (Y)
- net at R25.1, R26.1: now also U4.13 (-)
- net at R26.2: now also ADC2.7 (IN+), U4.14
- net at R20.2: now also ADC1.7 (IN+), U4.8
- net at R12.1, R20.1: now also U4.9 (-)
- net at C21.1, R18.1: now also U5.12 (+)
- net at C19.1, R14.1: now also U5.5 (+)
- net ~{CS_{1}}: now reaches ADC1.1 (~{CS})
- net ~{CS_{1}}: now also Q1.1 (G)
- net ADC_DATA_{1}: now reaches ADC1.2 (SDO)
- net ADC_DATA_{1}: now also JP7.1 (A)
- net ADC_CLK_{1}: now reaches ADC1.3 (SCLK)
- net ADC_CLK_{1}: now also JP8.1 (A)
- net at R22.2: now also JP5.2 (C), JP6.2 (B); no longer U20.13 (X)
- net at ADC2.1 (~{CS}): now also JP9.2 (C)
- net at ADC2.2 (SDO): now also JP7.2 (C)
- net at ADC2.3 (SCLK): now also JP8.2 (C)
- new net: JP9.3 (B), Q1.3 (D), R27.2
- new net: JP4.1 (A), U20.3 (Y)
- new net: U4.6 (-), U4.7
- new net: JP6.1 (A), U20.13 (X)
- new net ADC_CLK_{2}: JP8.3 (B)
- new net ADC_DATA_{2}: JP7.3 (B)
- new net ~{CS_{2}}: JP9.1 (A)
Other:
- moved on the sheet: ADC1, ADC2, C13, C15, C24, C26

Commit message: fix citace a uvod
Parts:
- removed C13, C15, C24, C26: 100n, Capacitor_SMD:C_0603_1608Metric_Pad1.08x0.95mm_HandSolder, symbol Device:C
- added TP10, TP11, TP12, TP13, TP14, TP5, TP6, TP7, TP8, TP9: TestPoint, Connector_Pin:Pin_D1.0mm_L10.0mm, symbol Connector:TestPoint
- JP4, JP6: footprint Connector_PinHeader_1.00mm:PinHeader_1x02_P1.00mm_Vertical -> Connector_PinHeader_2.54mm:PinHeader_1x02_P2.54mm_Vertical
Connections:
- net +1.65 V_{ref}: now also TP12.1
- net +3.3 V_{ref}: now also TP11.1
- net I_HighPass: now also TP7.1
- net I_LowPass: now also TP8.1
- net V_HighPass: now also TP5.1
- net V_LowPass: now also TP6.1
- net at ADC2.7 (IN+), R26.2, U4.14: now also TP14.1
- net at JP3.2 (C), JP4.2 (B), R24.2: now also TP10.1
- net at ADC1.7 (IN+), R20.2, U4.8: now also TP13.1
- net at JP5.2 (C), JP6.2 (B), R22.2: now also TP9.1
- net Sw_A: now reaches U20.10 (A)
- net Sw_B: now reaches U20.9 (B)
