File: Test_board_BAKALARKA/usb_power.kicad_sch (KiCad schematic)
At the start: 27 parts, among them J1 USB_C_Receptacle_USB2.0_16P, U1 LM27762, U3 HT75xx-1-SOT89

Commit message: fix citace a uvod
Parts:
- added TP15, TP16, TP17, TP18, TP19: TestPoint, Connector_Pin:Pin_D1.3mm_L11.0mm_LooseFit, symbol Connector:TestPoint
Connections:
- net GND: now also TP15.1, TP16.1, TP17.1, TP18.1, TP19.1
