File: Test_board_BAKALARKA/front_panel/front_panel.kicad_pcb (KiCad board)
At the start: 2 copper layers, 99.8 x 98 mm, 23 parts, among them SW1 SW_Push, SW10 SW_Push, SW11 SW_Push, SW12 SW_Push, SW13 SW_Push, SW14 SW_Push, SW15 SW_Push, SW16 SW_Push, SW17 SW_Push, SW18 SW_Push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

Commit message: front panel and test board ordered
Parts:
- added C1: 4u7, Capacitor_SMD:C_0805_2012Metric_Pad1.18x1.45mm_HandSolder, B.Cu at (88.8, 88.8)
- added D2: XINGLIGHT XL-1615RGBC-2812B-S, Snapeda:XINGLIGHT XL-1615RGBC-2812B-S, B.Cu at (95.0, 65.5)
- added D3: XINGLIGHT XL-1615RGBC-2812B-S, Snapeda:Flipped_XINGLIGHT XL-1615RGBC-2812B-S_1, B.Cu at (99.6, 63.2)
- added J1: Conn_01x10_Pin, PCM_JLCPCB:FFC_FPC_10pin_connector, B.Cu at (120.9, 90.2)
- added R2: 1k, Resistor_SMD:R_0603_1608Metric_Pad0.98x0.95mm_HandSolder, B.Cu at (101.2, 61.2)
- added R5: 1k, Resistor_SMD:R_0603_1608Metric_Pad0.98x0.95mm_HandSolder, B.Cu at (87.0, 89.8)
- added SW100: SW_SPST, Button_Switch_SMD:SW_SPST_CK_RS282G05A3, B.Cu at (107.4, 61.8)
- added SW101: SW_SPST, Button_Switch_SMD:SW_SPST_CK_RS282G05A3, B.Cu at (83.6, 93.4)
- added U2: ESP32-S3-WROOM-2, PCM_Espressif:ESP32-S3-WROOM-2, B.Cu at (100.5, 80.2)
- SW5, SW8: footprint PCM_JLCPCB:triangle -> PCM_JLCPCB:cap_touch_triangle
Connections:
- net Net-(SW1-Pad1) renamed /Touch array/Row 0
- net Net-(SW1-Pad2) renamed /Touch array/Col 0
- net Net-(SW10-Pad1) renamed /Touch array/Row 1
- net Net-(SW10-Pad2) renamed /Touch array/Col 2
- net Net-(SW11-Pad1) renamed /Touch array/Row 2
- net Net-(SW12-Pad1) renamed /Touch array/Row 3
- net Net-(SW13-Pad2) renamed /Touch array/Col 3
- net Net-(SW17-Pad2) renamed /Touch array/Col 4
- net Net-(SW21-Pad2) renamed /Touch array/Col 5
- net Net-(SW5-Pad2) renamed /Touch array/Col 1
Routing:
- net GND: track 0.00 -> 151.0 mm, vias 0 -> 31
- net +3V3: track 0.00 -> 111.6 mm, vias 0 -> 2
- net /Touch array/Col 5: track 8.80 -> 77.3 mm, vias 0 -> 1
- net /Touch array/Col 4: track 8.80 -> 65.7 mm, vias 0 -> 1
- net /Touch array/Col 3: track 8.80 -> 63.5 mm, vias 0 -> 1
- net Net-(J1-Pin_6): track 0.00 -> 48.5 mm, vias 0 -> 2
- net Net-(J1-Pin_7): track 0.00 -> 44.8 mm, vias 0 -> 2
- net /Touch array/Col 2: track 9.22 -> 47.6 mm, vias 0 -> 2
- net /Touch array/Row 0: track 79.1 -> 109.8 mm, vias 0 -> 1
- net Net-(SW100-B): track 0.00 -> 22.1 mm, vias 0 -> 3
- net Net-(SW101-B): track 0.00 -> 21.2 mm
- net sig3: track 0.00 -> 16.8 mm
- net /Touch array/Col 1: track 5.27 -> 21.6 mm, vias 0 -> 2
- net sig2: track 0.00 -> 16.2 mm
- net sig1: track 0.00 -> 15.9 mm
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- added copper zone on F.Cu, net GND
Other:
- outline, holes or cut-outs redrawn
