File: 2nd_prototype_LCRmeter/LEDs.kicad_sch (KiCad schematic)
At the start: 4 parts

Commit message: work on layout proto2
Parts:
- renumbered D21 to D15, D20 to D16, D19 to D17, R48 to R63
Changed lines of the file:
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@@
 		(on_board yes)
 		(dnp no)
-		(property "Reference" "R48"
+		(property "Reference" "R63"
 			(at 170.18 130.81 90)
 			(effects
@@
 			(project "LCR_Meter"
 				(path "/16346e7b-8abe-4c50-bf10-43609be2b1c5/fac0422f-7e79-4373-832c-9f162cf2289f"
-					(reference "R48")
+					(reference "R63")
 					(unit 1)
 				)
@@
 		(dnp no)
 		(fields_autoplaced yes)
-		(property "Reference" "#PWR03"
+		(property "Reference" "#PWR0140"
 			(at 184.15 104.14 0)
 			(effects
@@
 			(project "LCR_Meter"
 				(path "/16346e7b-8abe-4c50-bf10-43609be2b1c5/fac0422f-7e79-4373-832c-9f162cf2289f"
-					(reference "#PWR03")
+					(reference "#PWR0140")
 					(unit 1)
 				)
@@
 		(dnp no)
 		(fields_autoplaced yes)
-		(property "Reference" "#PWR0131"
+		(property "Reference" "#PWR0137"
 			(at 156.21 104.14 0)
 			(effects
@@
 			(project "LCR_Meter"
 				(path "/16346e7b-8abe-4c50-bf10-43609be2b1c5/fac0422f-7e79-4373-832c-9f162cf2289f"
-					(reference "#PWR0131")
+					(reference "#PWR0137")
 					(unit 1)
 				)
@@
 		(dnp no)
 		(fields_autoplaced yes)
-		(property "Reference" "#PWR04"
+		(property "Reference" "#PWR0141"
 			(at 184.15 121.92 0)
 			(effects
@@
 			(project "LCR_Meter"
 				(path "/16346e7b-8abe-4c50-bf10-43609be2b1c5/fac0422f-7e79-4373-832c-9f162cf2289f"
-					(reference "#PWR04")
+					(reference "#PWR0141")
 					(unit 1)
 				)
@@
 		(on_board yes)
 		(dnp no)
-		(property "Reference" "D19"
+		(property "Reference" "D17"
 			(at 172.72 101.6314 0)
 			(effects
@@
 			(project "LCR_Meter"
 				(path "/16346e7b-8abe-4c50-bf10-43609be2b1c5/fac0422f-7e79-4373-832c-9f162cf2289f"
-					(reference "D19")
+					(reference "D17")
 					(unit 1)
 				)
@@
 		(dnp no)
 		(fields_autoplaced yes)
-		(property "Reference" "#PWR0137"
+		(property "Reference" "#PWR0139"
 			(at 157.48 137.16 0)
 			(effects
@@
 			(project "LCR_Meter"
 				(path "/16346e7b-8abe-4c50-bf10-43609be2b1c5/fac0422f-7e79-4373-832c-9f162cf2289f"
-					(reference "#PWR0137")
+					(reference "#PWR0139")
 					(unit 1)
 				)
@@
 		(on_board yes)
 		(dnp no)
-		(property "Reference" "D20"
+		(property "Reference" "D16"
 			(at 179.07 133.35 0)
 			(effects
@@
 			(project "LCR_Meter"
 				(path "/16346e7b-8abe-4c50-bf10-43609be2b1c5/fac0422f-7e79-4373-832c-9f162cf2289f"
-					(reference "D20")
+					(reference "D16")
 					(unit 1)
 				)
@@
 		(on_board yes)
 		(dnp no)
-		(property "Reference" "D21"
+		(property "Reference" "D15"
 			(at 144.78 101.6314 0)
 			(effects
@@
 			(project "LCR_Meter"
 				(path "/16346e7b-8abe-4c50-bf10-43609be2b1c5/fac0422f-7e79-4373-832c-9f162cf2289f"
-					(reference "D21")
+					(reference "D15")
 					(unit 1)
 				)
@@
 		(dnp no)
 		(fields_autoplaced yes)
-		(property "Reference" "#PWR0132"
+		(property "Reference" "#PWR0138"
 			(at 156.21 121.92 0)
 			(effects
@@
 			(project "LCR_Meter"
 				(path "/16346e7b-8abe-4c50-bf10-43609be2b1c5/fac0422f-7e79-4373-832c-9f162cf2289f"
-					(reference "#PWR0132")
-					(unit 1)
-				)
+					(reference "#PWR0138")
+					(unit 1)
+				)
