File: 2nd_prototype_LCRmeter/PSU_USB.kicad_sch (KiCad schematic)
At the start: 21 parts, among them J5 USB_C_Receptacle_USB2.0_16P, U8 LM27762, U9 HT75xx-1-SOT89

Commit message: work on layout proto2
Parts:
- removed C2, C6, C8: 4.7u, Capacitor_SMD:C_0805_2012Metric_Pad1.18x1.45mm_HandSolder, symbol Device:C
- removed C51: 470u, Capacitor_THT:CP_Radial_D8.0mm_P3.80mm, symbol Device:C_Polarized
- added C13, C15, C16: 4.7u, Capacitor_SMD:C_0603_1608Metric, symbol Device:C
- added D18: LED, LED_SMD:LED_miniPLCC_2315_Handsoldering, symbol Device:LED
- added R64: 10k, Resistor_SMD:R_0603_1608Metric_Pad0.98x0.95mm_HandSolder, symbol Device:R
- added R65, R66: 5k1, Resistor_SMD:R_0603_1608Metric_Pad0.98x0.95mm_HandSolder, symbol Device:R
- C8: renamed from C1; footprint Capacitor_SMD:C_0805_2012Metric_Pad1.18x1.45mm_HandSolder -> Capacitor_SMD:C_0603_1608Metric
- C9: footprint Capacitor_SMD:C_0805_2012Metric_Pad1.18x1.45mm_HandSolder -> Capacitor_SMD:C_0603_1608Metric
- renumbered C3 to C10, C4 to C11, C5 to C12, C7 to C14, C12 to C18, C11 to C7, J5 to J4, R3 to R10, R4 to R11, R5 to R12, R1 to R8, R2 to R9, U8 to U2, U9 to U3
Connections:
- net +5V: now also C16.1; no longer C9.1
- net +5V_USB: now also C15.1, D18.2 (A), R64.2
- net -5V: now also C9.1
- net GND: now also C13.2, C15.2, C16.2, R65.1, R66.1; no longer U2.1 (PGOOD)
- net at U2.5 (CP): now also C13.1
- net at J4.A5 (CC1): now also R66.2
- net at J4.B5 (CC2): now also R65.2
- new net: D18.1 (K), R64.1, U2.1 (PGOOD)
- no-connect marks 4 -> 2
Other:
- moved on the sheet: C7, D1, J4, R8

Commit message: prod
Parts:
- added C29: 470u, Capacitor_Tantalum_SMD:CP_EIA-7343-30_AVX-N_HandSolder, symbol Device:C_Polarized
- C18, C7: footprint Capacitor_THT:CP_Radial_D8.0mm_P3.80mm -> Capacitor_Tantalum_SMD:CP_EIA-7343-30_AVX-N_HandSolder
Connections:
- net +5V: now also C29.1
- net GND: now also C29.2
Changed lines of the file:
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@@
+	)
+	(junction
+		(at 224.79 116.84)
+		(diameter 0)
+		(color 0 0 0 0)
 	)
 	(junction
@@
 	)
 	(symbol
+		(lib_id "Device:C_Polarized")
+		(at 224.79 120.65 0)
+		(unit 1)
+		(exclude_from_sim no)
+		(in_bom yes)
+		(on_board yes)
+		(dnp no)
+		(fields_autoplaced yes)
+		(property "Reference" "C29"
+			(at 228.6 118.4909 0)
+			(effects
+				(font
+					(size 1.27 1.27)
+				)
+				(justify left)
+			)
+		)
+		(property "Value" "470u"
+			(at 228.6 121.0309 0)
+			(effects
+				(font
+					(size 1.27 1.27)
+				)
+				(justify left)
+			)
+		)
+		(property "Footprint" "Capacitor_Tantalum_SMD:CP_EIA-7343-30_AVX-N_HandSolder"
+			(at 225.7552 124.46 0)
+			(effects
+				(font
+					(size 1.27 1.27)
+				)
+				(hide yes)
+			)
+		)
+		(property "Datasheet" "~"
+			(at 224.79 120.65 0)
+			(effects
+				(font
+					(size 1.27 1.27)
+				)
+				(hide yes)
+			)
+		)
+		(property "Description" "Polarized capacitor"
+			(at 224.79 120.65 0)
+			(effects
+				(font
+					(size 1.27 1.27)
+				)
+				(hide yes)
+			)
+		)
+		(pin "1"
+		)
+		(pin "2"
+		)
+		(instances
+			(project "V2_LCR_Meter"
+				(path "/16346e7b-8abe-4c50-bf10-43609be2b1c5/c4d4ab3e-37b0-40e2-997c-8f2441aa9b93"
+					(reference "C29")
+					(unit 1)
+				)
+			)
+		)
+	)
+	(symbol
 		(lib_id "Device:R")
 		(at 190.5 119.38 90)
@@
 	)
 	(symbol
+		(lib_id "power:GND")
+		(at 224.79 124.46 0)
+		(unit 1)
+		(exclude_from_sim no)
+		(in_bom yes)
+		(on_board yes)
+		(dnp no)
+		(fields_autoplaced yes)
+		(property "Reference" "#PWR066"
+			(at 224.79 130.81 0)
+			(effects
+				(font
+					(size 1.27 1.27)
+				)
+				(hide yes)
+			)
+		)
+		(property "Value" "GND"
+			(at 224.79 129.54 0)
+			(effects
+				(font
+					(size 1.27 1.27)
+				)
+			)
+		)
+		(property "Footprint" ""
+			(at 224.79 124.46 0)
+			(effects
+				(font
+					(size 1.27 1.27)
+				)
+				(hide yes)
+			)
+		)
+		(property "Datasheet" ""
+			(at 224.79 124.46 0)
+			(effects
+				(font
+					(size 1.27 1.27)
+				)
+				(hide yes)
+			)
+		)
+		(property "Description" "Power symbol creates a global label with name \"GND\" , ground"
+			(at 224.79 124.46 0)
+			(effects
+				(font
+					(size 1.27 1.27)
+				)
+				(hide yes)
+			)
+		)
+		(pin "1"
+		)
+		(instances
+			(project "V2_LCR_Meter"
+				(path "/16346e7b-8abe-4c50-bf10-43609be2b1c5/c4d4ab3e-37b0-40e2-997c-8f2441aa9b93"
+					(reference "#PWR066")
+					(unit 1)
+				)
+			)
+		)
+	)
+	(symbol
 		(lib_id "Device:C")
 		(at 180.34 140.97 0)
@@
 			)
 		)
-		(property "Footprint" "Capacitor_THT:CP_Radial_D8.0mm_P3.80mm"
+		(property "Footprint" "Capacitor_Tantalum_SMD:CP_EIA-7343-30_AVX-N_HandSolder"
 			(at 100.0252 124.46 0)
 			(effects
@@
 			)
 		)
-		(property "Footprint" "Capacitor_THT:CP_Radial_D8.0mm_P3.80mm"
+		(property "Footprint" "Capacitor_Tantalum_SMD:CP_EIA-7343-30_AVX-N_HandSolder"
 			(at 232.1052 139.7 0)
 			(effects
