File: 2nd_prototype_LCRmeter/frontend.kicad_sch (KiCad schematic)
At the start: 41 parts, among them J1 Conn_Coaxial, J2 Conn_Coaxial, J4 Conn_Coaxial, K1 Relay_DPDT, Q1 NX3008NBK, U14 CD74HC4052, U16 CD74HC4052, U17 INA823, U19 74LVC1G02, U2 TLV9154, U23 CD74HC4052, U4 LM393, U5 TLV9154

Commit message: work on layout proto2
Parts:
- removed JP4: SolderJumper_2_Open, Jumper:SolderJumper-2_P1.3mm_Open_TrianglePad1.0x1.5mm, symbol Jumper:SolderJumper_2_Open
- removed U2, U5: TLV9154, Package_SO:SOIC-14_3.9x8.7mm_P1.27mm, symbol Device:Opamp_Quad
- removed U4: LM393, Package_SO:SOIC-8_3.9x4.9mm_P1.27mm, symbol Comparator:LM393
- added C21, C24, C29, C30, C35, C36, C39, C40, C41, C42: 1u, Capacitor_SMD:C_0603_1608Metric_Pad1.08x0.95mm_HandSolder, symbol Device:C
- added C28, C32, C33, C34, C43, C44, C45: 330n, Capacitor_SMD:C_0603_1608Metric_Pad1.08x0.95mm_HandSolder, symbol Device:C
- added C47, C48, C49, C50: 100n, Capacitor_SMD:C_0603_1608Metric_Pad1.08x0.95mm_HandSolder, symbol Device:C
- added D2, D3, D4, D5, D6, D7, D8, D9: LED, LED_SMD:LED_miniPLCC_2315, symbol Device:LED
- added R13, R37: 1k, Resistor_SMD:R_0603_1608Metric_Pad0.98x0.95mm_HandSolder, symbol Device:R
- added R14, R39: 200k, Resistor_SMD:R_0603_1608Metric_Pad0.98x0.95mm_HandSolder, symbol Device:R
- added R15, R40: 100k, Resistor_SMD:R_0603_1608Metric_Pad0.98x0.95mm_HandSolder, symbol Device:R
- added R16, R41: 22k, Resistor_SMD:R_0603_1608Metric_Pad0.98x0.95mm_HandSolder, symbol Device:R
- added R17, R18, R19, R24, R25, R26, R27, R28, R29, R30, R31, R32, R42, R43, R44, R45, R46, R47, R48, R49, R50, R51, R52, R53, R54, R55: 10k, Resistor_SMD:R_0603_1608Metric_Pad0.98x0.95mm_HandSolder, symbol Device:R
- added TP1, TP10, TP2, TP3, TP4, TP5, TP6, TP7, TP8, TP9: TestPoint, Connector_Pin:Pin_D1.0mm_L10.0mm, symbol Connector:TestPoint
- added U10: TL072, Package_SO:SOIC-8_3.9x4.9mm_P1.27mm, symbol Amplifier_Operational:TL072
- added U12: INA823, Package_SO:SOIC-8_3.9x4.9mm_P1.27mm, symbol Amplifier_Instrumentation:INA128
- added U13, U5: CD74HC4052, Package_SO:TSSOP-16_4.4x5mm_P0.65mm, symbol Analog_Switch:CD4052B
- added U15: REF3033, Package_TO_SOT_SMD:SOT-23, symbol Reference_Voltage:REF3033
- added U4: OPA2192, Package_SO:SOIC-8_3.9x4.9mm_P1.27mm, symbol Device:Opamp_Dual
- added U7, U9: TL074, Package_SO:TSSOP-14_4.4x5mm_P0.65mm, symbol Amplifier_Operational:TL074
- C46: value 1u -> 330n
- J5: renamed from J2; now not fitted
- J8: renamed from J4; footprint Connector_Coaxial:BNC_Amphenol_B6252HB-NPP3G-50_Horizontal -> Snapeda:BNC_Gold
- J9: renamed from J1; footprint Connector_Coaxial:BNC_Amphenol_B6252HB-NPP3G-50_Horizontal -> Snapeda:BNC_Gold
- K1: footprint Relay_THT:Relay_CIT-J104D -> Relay_THT:Relay_DPDT_Finder_30.22
- gave numbers to parts that had none: 2
- renumbered C27 to C19, C28 to C20, C29 to C22, C30 to C23, C22 to C25, C34 to C27, C23 to C31, C33 to C37, C25 to C38, D7 to D10, D8 to D11, D9 to D12, D10 to D13, D2 to D14, R16 to R20, R19 to R21, R18 to R22, R17 to R23, R21 to R33, R22 to R34, R23 to R35, R24 to R36, R45 to R38, U16 to U11, U23 to U14, U19 to U16, U17 to U6, U14 to U8
Connections:
- net BNC_Shield is gone; now on net GND: J6.2 (Ext), J7.2 (Ext), J8.2 (Ext), J9.2 (Ext)
- net +3V3: now also R13.1, R37.1
- net +5V: now also C24.2, C29.2, C35.2, C40.2, C42.2, C47.2, U10.8 (V+), U12.7 (V+), U13.16 (VDD), U15.1 (IN), U4.8 (V+), U5.16 (VDD), U7.4 (V+), U9.4 (V+); no longer C46.2
- net -5V: now also C21.2, C30.2, C36.2, C39.2, C41.2, U10.4 (V-), U12.4 (V-), U13.7 (VEE), U4.4 (V-), U5.7 (VEE), U7.11 (V-), U9.11 (V-)
- net GND: now also C21.1, C24.1, C29.1, C30.1, C33.2, C35.1, C36.1, C39.1, C40.1, C41.1, C42.1, C45.2, C47.1, C48.1, C49.1, C50.1, D2.1 (K), D3.1 (K), D4.1 (K), D5.1 (K), D6.1 (K), D7.1 (K), D8.1 (K), D9.1 (K), R19.2, R29.2, R30.2, R44.2, R50.2, R51.2, R55.1, U12.5 (Ref), U13.6 (INH), U13.8 (VSS), U15.3 (GND), U4.6 (-), U5.6 (INH), U5.8 (VSS); no longer C46.1
- net I_ADC_AC: now also R53.2, TP9.1, U9.14
- net I_ADC_DC: now also R52.2, TP8.1, U9.7
- net Rg_1_A: now also U5.13 (X)
- net Rg_1_B: now also R14.2, R15.2, R16.2
- net SW_BYPASS_1_A: now also U4.1
- net Sig_IN: now also U4.3 (+)
- net V_ADC_AC: now also R32.2, TP4.1, U7.14
- net V_ADC_DC: now also R31.2, TP3.1, U7.7
- net at J6.1 (In): now also U6.2 (-)
- net at J7.1 (In): now also U6.3 (+)
- net at R33.2, R34.2, R35.2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: now also U12.3 (+), U4.7
- net at U11.3 (Y): now also U12.2 (-), U4.5 (+)
- net at U6.6: now also C28.2, R17.1
- net at U8.3 (Y): now also U4.2 (-)
- net I_Range_A renamed Shunt_Range_A
- net I_Range_B renamed Shunt_Range_B
- new net: C34.2, R17.2, R18.1
- new net: C46.2, R42.2, R43.1
- new net: C45.1, R43.2, U9.3 (+)
- new net: C44.1, R44.1, U9.10 (+)
- new net: C33.1, R18.2, U7.3 (+)
- new net: C28.1, C32.2, R24.1
- new net: R50.1, R52.1, U9.6 (-)
- new net: D4.2 (A), U5.2 (Y2)
- new net: R29.1, R31.1, U7.6 (-)
- new net: D7.2 (A), U13.5 (Y1)
- new net: C43.1, C44.2, R45.1
- new net: R30.1, R32.1, U7.13 (-)
- new net: R39.1, U13.14 (X1)
- new net: D9.2 (A), U13.4 (Y3)
- new net: R14.1, U5.14 (X1)
- new net: R51.1, R53.1, U9.13 (-)
- new net: D2.2 (A), U5.1 (Y0)
- new net: R27.1, R28.1, U7.12 (+)
- new net: R46.1, R47.1, U9.5 (+)
- new net: D5.2 (A), U5.4 (Y3)
- new net: R25.1, R26.1, U7.5 (+)
- new net: C43.2, R42.1, U12.6
- new net: R48.1, R49.1, U9.12 (+)
- new net: R41.1, U13.11 (X3)
- new net: R16.1, U5.11 (X3)
- new net: R37.2, U13.3 (Y)
- new net: C49.2, R54.1, R55.2, U10.3 (+)
- new net: R13.2, U5.3 (Y)
- new net: D3.2 (A), U5.5 (Y1)
- new net: C32.1, R19.1, U7.10 (+)
- new net: R40.1, U13.15 (X2)
- new net: D6.2 (A), U13.1 (Y0)
- new net: D8.2 (A), U13.2 (Y2)
- new net +1.65 V_{ref}: C50.2, R25.2, R27.2, R46.2, R48.2, TP10.1, U10.1, U10.2 (-)
- new net +3.3 V_{ref}: C48.2, R54.2, TP7.1, U15.2 (OUT)
- new net I_HighPass: R45.2, R49.2, TP5.1, U9.8, U9.9 (-)
- new net I_LowPass: C46.1, R47.2, TP6.1, U9.1, U9.2 (-)
- new net I_PGA_A: U13.10 (A)
- new net I_PGA_B: U13.9 (B)
- new net Rg_2_A: U12.8 (Rg), U13.13 (X)
- new net Rg_2_B: R39.2, R40.2, R41.2, U12.1 (Rg)
- new net V_HighPass: R24.2, R28.2, TP1.1, U7.8, U7.9 (-)
- new net V_LowPass: C34.1, R26.2, TP2.1, U7.1, U7.2 (-)
- new net V_PGA_A: U5.10 (A)
- new net V_PGA_B: U5.9 (B)
- no-connect marks 7 -> 9
Other:
- note added: "1.65V Offset"
- note added: "Current PGA"
- note added: "High pass"
- note added: "Low pass"
- note added: "Shunt range LED indicator"
- note added: "Shunt range relay bypass"
- note added: "Shunt range select"
- note added: "Voltage PGA"
- note added: "Voltage reference"
- note removed: "Range LED indicator"
- note removed: "Source output impedance selection"
- note removed: "Switch relay bypass - mitigate resistance for 100 Ohm range"
- moved on the sheet: C19, C20, C22, C23, C25, C26, D14, J6, J7, K1, Q1, U16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

Commit message: routing v2 work almost complete
Connections:
- net +5V: no longer D14.1 (K), K1.A1, U16.5 (VCC)
- net at U5.15 (X2): now also R15.1
- new net +5V_USB: D14.1 (K), K1.A1, U16.5 (VCC)
Changed lines of the file:
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@@
 	)
 	(junction
-		(at 351.79 35.56)
-		(diameter 0)
-		(color 0 0 0 0)
-	)
-	(junction
 		(at 97.79 36.83)
 		(diameter 0)
@@
 	)
 	(junction
+		(at 351.79 35.56)
+		(diameter 0)
+		(color 0 0 0 0)
+	)
+	(junction
 		(at 214.63 48.26)
 		(diameter 0)
@@
 	(wire
 		(pts
+			(xy 54.61 199.39) (xy 57.15 199.39)
+		)
+		(stroke
+			(width 0)
+			(type default)
+		)
+	)
+	(wire
+		(pts
 			(xy 54.61 212.09) (xy 58.42 212.09)
 		)
@@
 	(wire
 		(pts
+			(xy 351.79 33.02) (xy 351.79 35.56)
+		)
+		(stroke
+			(width 0)
+			(type default)
+		)
+	)
+	(wire
+		(pts
 			(xy 217.17 144.78) (xy 217.17 97.79)
 		)
@@
 	)
 	(symbol
+		(lib_id "power:+5V")
+		(at 351.79 33.02 0)
+		(unit 1)
+		(exclude_from_sim no)
+		(in_bom yes)
+		(on_board yes)
+		(dnp no)
+		(fields_autoplaced yes)
+		(property "Reference" "#PWR0113"
+			(at 351.79 36.83 0)
+			(effects
+				(font
+					(size 1.27 1.27)
+				)
+				(hide yes)
+			)
+		)
+		(property "Value" "+5V_USB"
+			(at 351.79 27.94 0)
+			(effects
+				(font
+					(size 1.27 1.27)
+				)
+			)
+		)
+		(property "Footprint" ""
+			(at 351.79 33.02 0)
+			(effects
+				(font
+					(size 1.27 1.27)
+				)
+				(hide yes)
+			)
+		)
+		(property "Datasheet" ""
+			(at 351.79 33.02 0)
+			(effects
+				(font
+					(size 1.27 1.27)
+				)
+				(hide yes)
+			)
+		)
+		(property "Description" "Power symbol creates a global label with name \"+5V\""
+			(at 351.79 33.02 0)
+			(effects
+				(font
+					(size 1.27 1.27)
+				)
+				(hide yes)
+			)
+		)
+		(pin "1"
+		)
+		(instances
+			(project "V2_LCR_Meter"
+				(path "/16346e7b-8abe-4c50-bf10-43609be2b1c5/846a19e8-f160-402c-9a0e-aa155abd6cf9"
+					(reference "#PWR0113")
+					(unit 1)
+				)
+			)
+		)
+	)
+	(symbol
 		(lib_id "power:GND")
 		(at 387.35 109.22 0)
@@
 	)
 	(symbol
+		(lib_id "power:+5V")
+		(at 323.85 45.72 0)
+		(unit 1)
+		(exclude_from_sim no)
+		(in_bom yes)
+		(on_board yes)
+		(dnp no)
+		(fields_autoplaced yes)
+		(property "Reference" "#PWR0149"
+			(at 323.85 49.53 0)
+			(effects
+				(font
+					(size 1.27 1.27)
+				)
+				(hide yes)
+			)
+		)
+		(property "Value" "+5V_USB"
+			(at 323.85 40.64 0)
+			(effects
+				(font
+					(size 1.27 1.27)
+				)
+			)
+		)
+		(property "Footprint" ""
+			(at 323.85 45.72 0)
+			(effects
+				(font
+					(size 1.27 1.27)
+				)
+				(hide yes)
+			)
+		)
+		(property "Datasheet" ""
+			(at 323.85 45.72 0)
+			(effects
+				(font
+					(size 1.27 1.27)
+				)
+				(hide yes)
+			)
+		)
+		(property "Description" "Power symbol creates a global label with name \"+5V\""
+			(at 323.85 45.72 0)
+			(effects
+				(font
+					(size 1.27 1.27)
+				)
+				(hide yes)
+			)
+		)
+		(pin "1"
+		)
+		(instances
+			(project "V2_LCR_Meter"
+				(path "/16346e7b-8abe-4c50-bf10-43609be2b1c5/846a19e8-f160-402c-9a0e-aa155abd6cf9"
+					(reference "#PWR0149")
+					(unit 1)
+				)
+			)
+		)
+	)
+	(symbol
 		(lib_id "power:GND")
 		(at 120.65 274.32 0)
@@
 	)
 	(symbol
-		(lib_id "power:+5V")
-		(at 351.79 35.56 0)
-		(unit 1)
-		(exclude_from_sim no)
-		(in_bom yes)
-		(on_board yes)
-		(dnp no)
-		(fields_autoplaced yes)
-		(property "Reference" "#PWR0117"
-			(at 351.79 39.37 0)
-			(effects
-				(font
-					(size 1.27 1.27)
-				)
-				(hide yes)
-			)
-		)
-		(property "Value" "+5V"
-			(at 351.79 30.48 0)
-			(effects
-				(font
-					(size 1.27 1.27)
-				)
-			)
-		)
-		(property "Footprint" ""
-			(at 351.79 35.56 0)
-			(effects
-				(font
-					(size 1.27 1.27)
-				)
-				(hide yes)
-			)
-		)
-		(property "Datasheet" ""
-			(at 351.79 35.56 0)
-			(effects
-				(font
-					(size 1.27 1.27)
-				)
-				(hide yes)
-			)
-		)
-		(property "Description" "Power symbol creates a global label with name \"+5V\""
-			(at 351.79 35.56 0)
-			(effects
-				(font
-					(size 1.27 1.27)
-				)
-				(hide yes)
-			)
-		)
-		(pin "1"
-		)
-		(instances
-			(project "LCR_Meter"
-				(path "/16346e7b-8abe-4c50-bf10-43609be2b1c5/846a19e8-f160-402c-9a0e-aa155abd6cf9"
-					(reference "#PWR0117")
-					(unit 1)
-				)
-			)
-		)
-	)
-	(symbol
 		(lib_id "Device:R")
 		(at 210.82 52.07 90)
@@
 					(unit 1)
 				)
-			)
-		)
-	)
-	(symbol
-		(lib_id "power:+5V")
-		(at 323.85 45.72 0)
-		(unit 1)
-		(exclude_from_sim no)
-		(in_bom yes)
-		(on_board yes)
-		(dnp no)
-		(fields_autoplaced yes)
-		(property "Reference" "#PWR0113"
-			(at 323.85 49.53 0)
-			(effects
-				(font
-					(size 1.27 1.27)
-				)
-				(hide yes)
-			)
-		)
-		(property "Value" "+5V"
-			(at 323.85 40.64 0)
-			(effects
-				(font
-					(size 1.27 1.27)
-				)
-			)
-		)
-		(property "Footprint" ""
-			(at 323.85 45.72 0)
-			(effects
-				(font
-					(size 1.27 1.27)
-				)
-				(hide yes)
-			)
-		)
-		(property "Datasheet" ""
-			(at 323.85 45.72 0)
-			(effects
-				(font
-					(size 1.27 1.27)
-				)
-				(hide yes)
-			)
-		)
-		(property "Description" "Power symbol creates a global label with name \"+5V\""
-			(at 323.85 45.72 0)
-			(effects
-				(font
-					(size 1.27 1.27)
-				)
-				(hide yes)
-			)
-		)
-		(pin "1"
-		)
-		(instances
-			(project "LCR_Meter"
-				(path "/16346e7b-8abe-4c50-bf10-43609be2b1c5/846a19e8-f160-402c-9a0e-aa155abd6cf9"
-					(reference "#PWR0113")
-					(unit 1)
-				)

Commit message: finished with offset amps
Parts:
- R14, R39: value 200k -> 100k
- R15, R40: value 100k -> 25k
- R16: value 22k -> 11k
- R41: value 22k -> 100k
Connections:
- net GND: now also U10.5 (+)
- net at U10.6 (-): now also U10.7
Changed lines of the file:
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@@
 	(wire
 		(pts
+			(xy 387.35 132.08) (xy 381 132.08)
+		)
+		(stroke
+			(width 0)
+			(type default)
+		)
+	)
+	(wire
+		(pts
 			(xy 66.04 212.09) (xy 69.85 212.09)
 		)
@@
 	(wire
 		(pts
+			(xy 402.59 134.62) (xy 402.59 142.24)
+		)
+		(stroke
+			(width 0)
+			(type default)
+		)
+	)
+	(wire
+		(pts
 			(xy 259.08 208.28) (xy 259.08 210.82)
 		)
@@
 	(wire
 		(pts
+			(xy 384.81 137.16) (xy 387.35 137.16)
+		)
+		(stroke
+			(width 0)
+			(type default)
+		)
+	)
+	(wire
+		(pts
 			(xy 101.6 36.83) (xy 97.79 36.83)
 		)
@@
 	(wire
 		(pts
+			(xy 402.59 142.24) (xy 384.81 142.24)
+		)
+		(stroke
+			(width 0)
+			(type default)
+		)
+	)
+	(wire
+		(pts
 			(xy 88.9 52.07) (xy 85.09 52.07)
 		)
@@
 	(wire
 		(pts
+			(xy 384.81 142.24) (xy 384.81 137.16)
+		)
+		(stroke
+			(width 0)
+			(type default)
+		)
+	)
+	(wire
+		(pts
 			(xy 261.62 226.06) (xy 257.81 226.06)
 		)
@@
 	(wire
 		(pts
+			(xy 381 132.08) (xy 381 133.35)
+		)
+		(stroke
+			(width 0)
+			(type default)
+		)
+	)
+	(wire
+		(pts
 			(xy 308.61 87.63) (xy 318.77 87.63)
 		)
@@
 			)
 		)
-		(property "Value" "200k"
+		(property "Value" "100k"
 			(at 262.636 208.28 90)
 			(effects
@@
 			)
 		)
-		(property "Value" "200k"
+		(property "Value" "100k"
 			(at 70.866 196.85 90)
 			(effects
@@
 	(symbol
 		(lib_id "power:GND")
+		(at 381 133.35 0)
+		(unit 1)
+		(exclude_from_sim no)
+		(in_bom yes)
+		(on_board yes)
+		(dnp no)
+		(fields_autoplaced yes)
+		(property "Reference" "#PWR0117"
+			(at 381 139.7 0)
+			(effects
+				(font
+					(size 1.27 1.27)
+				)
+				(hide yes)
+			)
+		)
+		(property "Value" "GND"
+			(at 381 138.43 0)
+			(effects
+				(font
+					(size 1.27 1.27)
+				)
+			)
+		)
+		(property "Footprint" ""
+			(at 381 133.35 0)
+			(effects
+				(font
+					(size 1.27 1.27)
+				)
+				(hide yes)
+			)
+		)
+		(property "Datasheet" ""
+			(at 381 133.35 0)
+			(effects
+				(font
+					(size 1.27 1.27)
+				)
+				(hide yes)
+			)
+		)
+		(property "Description" "Power symbol creates a global label with name \"GND\" , ground"
+			(at 381 133.35 0)
+			(effects
+				(font
+					(size 1.27 1.27)
+				)
+				(hide yes)
+			)
+		)
+		(pin "1"
+		)
+		(instances
+			(project "V2_LCR_Meter"
+				(path "/16346e7b-8abe-4c50-bf10-43609be2b1c5/846a19e8-f160-402c-9a0e-aa155abd6cf9"
+					(reference "#PWR0117")
+					(unit 1)
+				)
+			)
+		)
+	)
+	(symbol
+		(lib_id "power:GND")
 		(at 261.62 59.69 0)
 		(unit 1)
@@
 			)
 		)
-		(property "Value" "22k"
+		(property "Value" "100k"
 			(at 262.636 213.106 90)
 			(effects
@@
 			)
 		)
-		(property "Value" "22k"
+		(property "Value" "11k"
 			(at 70.866 201.676 90)
 			(effects
@@
 			)
 		)
-		(property "Value" "100k"
+		(property "Value" "25k"
 			(at 262.636 210.82 90)
 			(effects
@@
 			)
 		)
-		(property "Value" "100k"
+		(property "Value" "25k"
 			(at 70.866 199.39 90)
 			(effects

Commit message: finished final final_2
Parts:
- removed C29, C30: 1u, Capacitor_SMD:C_0603_1608Metric_Pad1.08x0.95mm_HandSolder, symbol Device:C
- removed J5: Conn_Coaxial, Connector_Coaxial:BNC_Amphenol_B6252HB-NPP3G-50_Horizontal, symbol Connector:Conn_Coaxial
- removed R25, R26, R27, R28, R29, R30, R31, R32, R46, R47, R48, R49, R50, R51, R52, R53: 10k, Resistor_SMD:R_0603_1608Metric_Pad0.98x0.95mm_HandSolder, symbol Device:R
- removed TP3, TP4, TP8, TP9: TestPoint, Connector_Pin:Pin_D1.0mm_L10.0mm, symbol Connector:TestPoint
- removed U9: TL074, Package_SO:TSSOP-14_4.4x5mm_P0.65mm, symbol Amplifier_Operational:TL074
- C28, C32, C33, C34, C43, C44, C45, C46: value 330n -> 100n
- R17, R18, R19, R24, R42, R43, R44, R45: value 10k -> 100k
Connections:
- net I_HighPass is gone; now on net I_ADC_AC: R45.2, TP5.1
- net I_LowPass is gone; now on net I_ADC_DC: C46.1, TP6.1
- net V_LowPass is gone; now on net V_ADC_DC: C34.1, TP2.1, U7.1, U7.2 (-)
- net +1.65 V_{ref}: now also U12.5 (Ref), U6.5 (Ref)
- net GND: no longer U12.5 (Ref), U6.5 (Ref)
- net I_ADC_AC: now also U7.13 (-), U7.14
- net I_ADC_DC: now also U7.8, U7.9 (-)
- net V_ADC_AC: now also R24.2, TP1.1, U7.6 (-), U7.7; no longer U7.14
- net V_ADC_DC: no longer U7.7
- net at C45.1, R43.2: now also U7.10 (+)
- net at C44.1, R44.1: now also U7.12 (+)
- net at U7.5 (+): now also C32.1, R19.1
- removed net V_HighPass: R24.2, TP1.1, U7.8, U7.9 (-)
Other:
- note added: "15,9 Hz Cutoff"
- note removed: "1.65V Offset"
- moved on the sheet: C21, C22, C23, C24, C28, C32, C33, C34, C39, C40, C41, C42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
