File: 2nd_prototype_LCRmeter/frontend.kicad_sch (KiCad schematic)
At the start: 94 parts, among them J6 Conn_Coaxial, J7 Conn_Coaxial, J8 Conn_Coaxial, J9 Conn_Coaxial, K1 Relay_DPDT, Q1 NX3008NBK, U10 TL072, U11 CD74HC4052, U12 INA823, U13 CD74HC4052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

Commit message: update
Changed lines of the file:
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@@
-		)
-	)
-	(text "Chyba! "
-		(exclude_from_sim no)
-		(at 187.96 97.79 0)
-		(effects
-			(font
-				(size 7.62 7.62)
-				(thickness 1.524)
-				(bold yes)
-				(color 245 255 0 1)
-			)
 		)
 	)
