File: 2nd_prototype_LCRmeter/V2_LCR_Meter.kicad_sch (KiCad schematic)
At the start: 17 parts, among them J6 IDC 2x5, J7 Display OLED, SW1 SW_SPST

Commit message: work on layout proto2
Parts:
- added C1, C2: 20p, Capacitor_SMD:C_0603_1608Metric_Pad1.08x0.95mm_HandSolder, symbol Device:C_Small
- added TP11, TP12, TP13, TP14, TP15, TP16, TP17, TP18, TP19: TestPoint, Connector_Pin:Pin_D1.0mm_L10.0mm, symbol Connector:TestPoint
- added Y1: 8MHz, Crystal:Crystal_HC49-U_Vertical, symbol Device:Crystal
- J1: renamed from J?; footprint Connector_PinHeader_2.54mm:PinHeader_1x04_P2.54mm_Vertical -> Connector_PinHeader_2.54mm:PinHeader_1x04_P2.54mm_Vertical_SMD_Pin1Left
- JP1: renamed from JP2; footprint Connector_PinHeader_2.54mm:PinHeader_1x03_P2.54mm_Vertical -> Connector_PinHeader_2.54mm:PinHeader_1x03_P2.54mm_Vertical_SMD_Pin1Left
- gave numbers to parts that had none: 7
- renumbered C10 to C3, J7 to J2, J6 to J3, R7 to R1, R43 to R2, R44 to R5
Connections:
- net +3V3: now also U1.1 (VBAT), U1.9 (VDDA), TP14.1
- net +5V: now also TP11.1
- net -5V: now also TP12.1
- net GND: now also J3.2 (Pin_2), U1.8 (VSSA), C1.2, C2.2, TP13.1, TP15.1, TP16.1, TP17.1, TP18.1, TP19.1
- net I_PGA_A: now also U1.21 (PB10)
- net I_PGA_B: now also U1.22 (PB11)
- net LEDs/LED_1: now also U1.28 (PB15)
- net LEDs/RGB_Data: now also U1.27 (PB14)
- net MISO: now also U1.40 (PB4)
- net MOSI: now also U1.41 (PB5)
- net NSS: now also U1.38 (PA15)
- net SCK: now also U1.39 (PB3)
- net UART_RX: now also J3.4 (Pin_4)
- net UART_TX: now also J3.7 (Pin_7)
- net V_PGA_A: now also U1.25 (PB12)
- net V_PGA_B: now also U1.26 (PB13)
- net at R3.1: now also JP1.3 (B); no longer JP1.1 (A)
- net at R1.2: now also JP1.1 (A); no longer JP1.3 (B)
- net GPIO_PA0: now reaches U1.10 (PA0)
- net GPIO_PA0: now also J3.3 (Pin_3)
- net Shunt_Range_A: now reaches U1.45 (PB8)
- net Shunt_Range_B: now reaches U1.46 (PB9)
- net at U1.5 (PD0): now also C1.1, Y1.2
- net at U1.6 (PD1): now also C2.1, Y1.1
- no-connect marks 0 -> 3
Other:
- note added: "Add-on connect"
- note added: "I^{2}C Pullup"
- note added: "Net color tags"
- note added: "OLED Connect"
- note added: "ST-Link Connect"
- note removed: "ST-Link connect"
- moved on the sheet: J2, J3, JP1, R1, R2, R3, R5, R6, SW1

Commit message: routing v2 work almost complete
Connections:
- net Analog frontend/I_ADC_AC: now also U1.14 (PA4); no longer U1.13 (PA3)
- net Analog frontend/I_ADC_DC: now also U1.13 (PA3); no longer U1.11 (PA1)
- net Analog frontend/V_ADC_AC: now also U1.11 (PA1); no longer U1.14 (PA4)
Changed lines of the file:
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@@
 	(wire
 		(pts
+			(xy 107.95 58.42) (xy 123.19 58.42)
+		)
+		(stroke
+			(width 0)
+			(type default)
+		)
+	)
+	(wire
+		(pts
 			(xy 48.26 45.72) (xy 50.8 45.72)
 		)
@@
 	(wire
 		(pts
+			(xy 107.95 55.88) (xy 123.19 55.88)
+		)
+		(stroke
+			(width 0)
+			(type default)
+		)
+	)
+	(wire
+		(pts
 			(xy 25.4 27.94) (xy 35.56 27.94)
 		)
@@
 	(wire
 		(pts
-			(xy 105.41 21.59) (xy 115.57 21.59)
+			(xy 107.95 50.8) (xy 123.19 50.8)
 		)
 		(stroke
@@
 	(wire
 		(pts
-			(xy 107.95 63.5) (xy 180.34 63.5)
+			(xy 105.41 21.59) (xy 115.57 21.59)
 		)
 		(stroke
@@
 	(wire
 		(pts
-			(xy 157.48 144.78) (xy 162.56 144.78)
+			(xy 107.95 63.5) (xy 180.34 63.5)
 		)
 		(stroke
@@
 	(wire
 		(pts
-			(xy 179.07 55.88) (xy 179.07 60.96)
+			(xy 157.48 144.78) (xy 162.56 144.78)
 		)
 		(stroke
@@
 	(wire
 		(pts
-			(xy 107.95 53.34) (xy 123.19 53.34)
+			(xy 179.07 55.88) (xy 179.07 60.96)
 		)
 		(stroke
@@
 	(wire
 		(pts
-			(xy 107.95 58.42) (xy 123.19 58.42)
-		)
-		(stroke
-			(width 0)
-			(type default)
-		)
-	)
-	(wire
-		(pts
 			(xy 95.25 40.64) (xy 95.25 36.83)
 		)
@@
 	(wire
 		(pts
-			(xy 107.95 50.8) (xy 123.19 50.8)
-		)
-		(stroke
-			(width 0)
-			(type default)
-		)
-	)
-	(wire
-		(pts
 			(xy 107.95 76.2) (xy 201.93 76.2)
 		)
@@
 	(wire
 		(pts
+			(xy 107.95 53.34) (xy 123.19 53.34)
+		)
+		(stroke
+			(width 0)
+			(type default)
+		)
+	)
+	(wire
+		(pts
 			(xy 16.51 45.72) (xy 20.32 45.72)
 		)
@@
 	(wire
 		(pts
-			(xy 107.95 55.88) (xy 123.19 55.88)
-		)
-		(stroke
-			(width 0)
-			(type default)
-		)
-	)
-	(wire
-		(pts
 			(xy 275.59 135.89) (xy 266.7 135.89)
 		)
@@
 		)
 		(pin "I_ADC_DC" output
-			(at 123.19 50.8 180)
+			(at 123.19 55.88 180)
 			(effects
 				(font
@@
 		)
 		(pin "V_ADC_AC" output
-			(at 123.19 58.42 180)
+			(at 123.19 50.8 180)
 			(effects
 				(font
@@
 		)
 		(pin "I_ADC_AC" output
-			(at 123.19 55.88 180)
+			(at 123.19 58.42 180)
 			(effects
 				(font
