File: 2nd_prototype_LCRmeter/V2_LCR_Meter.kicad_pcb (KiCad board)
At the start: 6 copper layers, 99.8 x 99.8 mm, 209 parts, among them J1 ST-Link, J2 Display OLED, J3 IDC 2x5, J4 USB_C_Receptacle_USB2.0_16P, J6 Conn_Coaxial, J7 Conn_Coaxial, J8 Conn_Coaxial, J9 Conn_Coaxial, K1 Relay_DPDT, Q1 NX3008NBK, SW1 SW_SPST, U1 STM32F103C8Tx, U10 TL072, U11 CD74HC4052, U12 INA823, U13 CD74HC4052, U14 CD74HC4052, U15 REF3033, U16 74LVC1G02, U18 TL074, U19 MCP4561-502E_MS, U2 LM27762, U20 AD9837, U3 HT75xx-1-SOT89, U4 OPA2192, U5 CD74HC4052, U6 INA823, U7 TL074, U8 CD74HC4052, X1 SG-210STF, Y1 8MHz

Commit message: prod
Parts:
- added C29: 470u, Capacitor_Tantalum_SMD:CP_EIA-7343-30_AVX-N_HandSolder, F.Cu at (256.0, 39.2)
- added G***: LOGO, LOGO, F.Cu at (182.0, 72.8)
- added kibuzzard-69B032D8: G***, kibuzzard-69B032D8, F.Cu at (186.6, 31.0)
- added kibuzzard-69B032F6: G***, kibuzzard-69B032F6, F.Cu at (211.2, 26.0)
- added kibuzzard-69B03341: G***, kibuzzard-69B03341, F.Cu at (199.8, 25.6)
- added kibuzzard-69B03368: G***, kibuzzard-69B03368, F.Cu at (194.8, 30.6)
- added kibuzzard-69B03378: G***, kibuzzard-69B03378, F.Cu at (204.8, 30.6)
- C18, C7: footprint Capacitor_THT:CP_Radial_D8.0mm_P3.80mm -> Capacitor_Tantalum_SMD:CP_EIA-7343-30_AVX-N_HandSolder
- R1, R3: moved to B.Cu
- moved C18 13.2 mm to (256.0, 44.4), turned to 0 degrees
- moved C7 2.41 mm to (241.8, 34.2), turned to 0 degrees
Routing:
- net GND: track 139.0 -> 121.0 mm, vias 78 -> 81
- net +5V: track 13.4 -> 26.0 mm, vias 13 -> 14
- net -5V: track 12.2 -> 17.8 mm, vias 12 -> 13
- net +5V_USB: track 180.7 -> 179.9 mm
- net Net-(JP1-B): vias 0 -> 1
- net Net-(JP1-A): vias 0 -> 1
