File: Final_schematic/frontend.kicad_sch (KiCad schematic)
At the start: 94 parts, among them J6 Conn_Coaxial, J7 Conn_Coaxial, J8 Conn_Coaxial, J9 Conn_Coaxial, K1 Relay_DPDT, Q1 NX3008NBK, U10 TL072, U11 CD74HC4052, U12 INA823, U13 CD74HC4052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

Commit message: Removed obsolete PDF files and updated LaTeX documents with new sections and references.
Parts:
- removed C28, C32, C33, C34, C43, C44, C45, C46: 100n, Capacitor_SMD:C_0603_1608Metric_Pad1.08x0.95mm_HandSolder, symbol Device:C
- removed R17, R18, R19, R24, R42, R43, R44, R45: 100k, Resistor_SMD:R_0603_1608Metric_Pad0.98x0.95mm_HandSolder, symbol Device:R
- removed TP1, TP2, TP5, TP6: TestPoint, Connector_Pin:Pin_D1.0mm_L10.0mm, symbol Connector:TestPoint
- removed unit 2 of U10
- removed unit 1 of U7
- removed unit 3 of U7
- removed unit 2 of U7
- removed unit 4 of U7
Connections:
- net GND: now also U4.5 (+); no longer U4.6 (-)
- net I_ADC_AC: now also U12.6
- net V_ADC_AC: now also U6.6
- net at U11.3 (Y), U12.2 (-): now also U4.6 (-); no longer U4.5 (+)
Other:
- note added: "I-U převodník"
- note added: "LED indikátor bočníku"
- note added: "Napájení operačních zesilovačů"
- note added: "Napěťová reference"
- note added: "Napěťový zesilovač"
- note added: "Selekce bočníku"
- note added: "Spínač bočníku s nízkou hodnotou"
- note added: "Toto schéma obsahuje opravy z produkčního schématu V2. Zbytečné prvky jsou vynechány pro jednoduchost."
- note removed: "15,9 Hz Cutoff"
- note removed: "Chyba!"
- note removed: "High pass"
- note removed: "Low pass"
- note removed: "Shunt range LED indicator"
- note removed: "Shunt range relay bypass"
- note removed: "Shunt range select"
- note removed: "Voltage PGA"
- note removed: "Voltage reference"
- moved on the sheet: C19, C20, C25, C26, C35, C36, C39, C40, C41, C47, C48, C49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
