File: schemata_kicad/XOR_phase.kicad_sch (KiCad schematic)
At the start: 7 parts, among them U10 VSIN, U7 XOR, U9 VSIN

Commit message: pridane nastaveni dc offsetu do zdroje a neco ke vzorkovani
Connections:
- net at U7.: now also U11.; no longer U8.
- new net: U7., U8.

Commit message: update
Parts:
- U11, U8: value ~ -> (none)
Connections:
- net at U7.: now also U11.; no longer U8.
- new net: U7., U8.

Commit message: 4wire a dalsi
Connections:
- net at U7.: now also U11.; no longer U8.
- new net: U7., U8.
