File: schemata_kicad/amplitude.kicad_sch (KiCad schematic)
At the start: 7 parts, among them U13 VSIN

Commit message: pridane nastaveni dc offsetu do zdroje a neco ke vzorkovani
Parts:
- renumbered TP1 to TP?, sdf to sdf?
Changed lines of the file:
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@@
 		(on_board yes)
 		(dnp no)
-		(property "Reference" "sdf"
+		(property "Reference" "sdf?"
 			(at 59.69 43.1799 0)
 			(effects
@@
 		)
 		(pin ""
-		)
-		(instances
-			(project ""
-				(path "/ba5b7f3f-bcc2-4274-bf72-d951c4da15c7/cc843ba0-d1bd-4c35-8f2d-0fd5113ded5b"
-					(reference "sdf")
-					(unit 1)
-				)
-			)
 		)
 	)
@@
 		(dnp no)
 		(fields_autoplaced yes)
-		(property "Reference" "TP1"
+		(property "Reference" "TP?"
 			(at 112.5221 39.37 0)
 			(effects
@@
 		(pin "1"
 		)
-		(instances
-			(project ""
-				(path "/ba5b7f3f-bcc2-4274-bf72-d951c4da15c7/cc843ba0-d1bd-4c35-8f2d-0fd5113ded5b"
-					(reference "TP1")
-					(unit 1)
-				)
-			)
-		)
-	)
+	)

Commit message: update
Parts:
- U12: value ~ -> (none)
