File: schemata_kicad/wheatstone.kicad_sch (KiCad schematic)
At the start: 5 parts, among them U3 VSIN

Commit message: prace na prototypu a tak
Parts:
- renumbered U3 to U?, Z6 to Z2, Zx1 to Zx
Changed lines of the file:
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@@
 		(on_board yes)
 		(dnp no)
-		(property "Reference" "Z6"
+		(property "Reference" "Z2"
 			(at 128.778 52.07 0)
 			(effects
@@
 		)
 		(instances
+			(project "wheatstone"
+				(path "/71305d32-c10f-4c05-8337-91cd088b5d4d"
+					(reference "Z2")
+					(unit 1)
+				)
+			)
 			(project ""
 				(path "/ba5b7f3f-bcc2-4274-bf72-d951c4da15c7/e39c6ceb-98aa-46f9-8e7d-c134b310cc1c"
@@
 		(on_board yes)
 		(dnp no)
-		(property "Reference" "Zx1"
+		(property "Reference" "Zx"
 			(at 127.762 66.802 90)
 			(effects
@@
 		)
 		(instances
+			(project "wheatstone"
+				(path "/71305d32-c10f-4c05-8337-91cd088b5d4d"
+					(reference "Zx")
+					(unit 1)
+				)
+			)
 			(project ""
 				(path "/ba5b7f3f-bcc2-4274-bf72-d951c4da15c7/e39c6ceb-98aa-46f9-8e7d-c134b310cc1c"
@@
 		)
 		(instances
+			(project "wheatstone"
+				(path "/71305d32-c10f-4c05-8337-91cd088b5d4d"
+					(reference "Z1")
+					(unit 1)
+				)
+			)
 			(project "schemata"
 				(path "/ba5b7f3f-bcc2-4274-bf72-d951c4da15c7/e39c6ceb-98aa-46f9-8e7d-c134b310cc1c"
@@
 		)
 		(instances
+			(project "wheatstone"
+				(path "/71305d32-c10f-4c05-8337-91cd088b5d4d"
+					(reference "Z3")
+					(unit 1)
+				)
+			)
 			(project "schemata"
 				(path "/ba5b7f3f-bcc2-4274-bf72-d951c4da15c7/e39c6ceb-98aa-46f9-8e7d-c134b310cc1c"
@@
 		(dnp no)
 		(fields_autoplaced yes)
-		(property "Reference" "U3"
+		(property "Reference" "U?"
 			(at 102.87 67.1801 0)
 			(effects
@@
 		)
 		(instances
+			(project "wheatstone"
+				(path "/71305d32-c10f-4c05-8337-91cd088b5d4d"
+					(reference "U?")
+					(unit 1)
+				)
+			)
 			(project "schemata"
 				(path "/ba5b7f3f-bcc2-4274-bf72-d951c4da15c7/e39c6ceb-98aa-46f9-8e7d-c134b310cc1c"
@@
 		)
 	)
+	(sheet_instances
+		(path "/"
+			(page "1")
+		)
+	)
+	(embedded_fonts no)
 )

Commit message: update
Parts:
- Z6: renamed from Z2; value ~ -> (none)
- gave numbers to parts that had none: 1
- renumbered Zx to Zx1
